File: CM5-AI-Cam-CopperPilot.kicad_sch (KiCad schematic)
At the start: 90 parts, among them J1 IMX219_30P, J2 USB_A_Vertical, Q1 DMG1012T, Q2 DMG1012T, U1 RT9193-28GB, U2 RT9193-18GB, U3 RT9013-12, U4 STMPS2171STR, U5 MP1658GTF-Z, U6 FSUSB42MX, U7 STMPS2171STR, U8 STMPS2171STR, X1 OSC_24MHz

Commit message: fix(hardware): separate 100R MIPI/HDMI and 90R USB netclasses and resolve BOM/SCH/PCB review defects
- Assign HighSpeed_100R (100 Ohm diff: W=0.127mm, S=0.150mm -> 100.1 Ohm on JLC06161H-7628 stripline / 98.3 Ohm on JLC06161H-3313 microstrip) to MIPI CSI-2, MIPI DSI, and HDMI TMDS pairs, and HighSpeed_90R (90 Ohm diff: W=0.180mm, S=0.150mm -> 89.6 Ohm stripline / 88.7 Ohm microstrip) to USB 2.0 pairs in .kicad_pro, .kicad_pcb, and .kicad_dru.
- Synchronize .kicad_pcb stackup dielectric parameters with JLCPCB JLC06161H-7628 (0.2104mm prepreg, 0.4000mm core, er=4.6).
- Restore C20 on 24 MHz camera MCLK from 0.1uF (72.3 kHz cutoff) to 10pF (C32949, fc=723 MHz) and correct LCSC codes for R20 (C25803 61.9k), U3 (C47773 1.2V LDO), U1 (C15075 2.8V LDO), U5 (C2960187 MP1658GTF-Z), HDMI1 (C424662), L1-L3 (C110443), C21 (C1534 330pF), and U6 (FSUSB42UMX C11145).
- Exclude DNP straps R31, R32, R33 from BOM and CPL (--exclude-dnp) so CM5 Wi-Fi and Bluetooth remain enabled.
- Repair missing pad coordinates in CM5.pretty/R_0402_1005Metric.kicad_mod, TF1 SMD attribute, and 3D model  paths, and expand PyTest suite to 29 tests.

Co-Authored-By: CopperPilot <noreply@copperpilot.ai>
Parts:
- C10, C14, C3: value 100nF -> 0.1uF
- C20: value 0.1uF -> 10pF; LCSC C1525 -> C32949
- C21: LCSC C1547 -> C1534
- HDMI1: LCSC C2013978 -> C424662
- L1, L2, L3: LCSC C49073870 -> C110443
- R20: LCSC C25916 -> C25803
- U1: LCSC C114059 -> C15075
- U3: LCSC C7434207 -> C47773
- U5: LCSC C2837379 -> C2960187
- U6: value FSUSB42MX -> FSUSB42UMX
Changed lines of the file:
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@@
 			(effects (font (size 1.27 1.27)) (hide yes))
 		)
-		(property "LCSC" "C2837379"
+		(property "LCSC" "C2960187"
 			(at 250.1900 66.0400 0)
 			(effects (font (size 1.27 1.27)) (hide yes))
@@
 			(effects (font (size 1.27 1.27)) (hide yes))
 		)
-		(property "LCSC" "C1547"
+		(property "LCSC" "C1534"
 			(at 288.2900 50.8000 0)
 			(effects (font (size 1.27 1.27)) (hide yes))
@@
 			(effects (font (size 1.27 1.27)) (hide yes))
 		)
-		(property "LCSC" "C25916"
+		(property "LCSC" "C25803"
 			(at 288.2900 82.5500 0)
 			(effects (font (size 1.27 1.27)) (hide yes))
@@
 			(effects (font (size 1.27 1.27)))
 		)
-		(property "Value" "FSUSB42MX"
+		(property "Value" "FSUSB42UMX"
 			(at 454.6600 279.4000 0)
 			(effects (font (size 1.27 1.27)))
@@
 			(effects (font (size 1.27 1.27)) (hide yes))
 		)
-		(property "LCSC" "C49073870"
+		(property "LCSC" "C110443"
 			(at 350.5200 151.1300 0)
 			(effects (font (size 1.27 1.27)) (hide yes))
@@
 			(effects (font (size 1.27 1.27)) (hide yes))
 		)
-		(property "LCSC" "C49073870"
+		(property "LCSC" "C110443"
 			(at 350.5200 166.3700 0)
 			(effects (font (size 1.27 1.27)) (hide yes))
@@
 			(effects (font (size 1.27 1.27)) (hide yes))
 		)
-		(property "LCSC" "C49073870"
+		(property "LCSC" "C110443"
 			(at 350.5200 181.6100 0)
 			(effects (font (size 1.27 1.27)) (hide yes))
@@
 			(effects (font (size 1.27 1.27)) (hide yes))
 		)
-		(property "LCSC" "C114059"
+		(property "LCSC" "C15075"
 			(at 335.2800 231.1400 0)
 			(effects (font (size 1.27 1.27)) (hide yes))
@@
 			(effects (font (size 1.27 1.27)))
 		)
-		(property "Value" "100nF"
+		(property "Value" "0.1uF"
 			(at 283.9720 196.8500 0)
 			(effects (font (size 1.27 1.27)))
@@
 			(effects (font (size 1.27 1.27)))
 		)
-		(property "Value" "100nF"
+		(property "Value" "0.1uF"
 			(at 286.5120 240.0300 0)
 			(effects (font (size 1.27 1.27)))
@@
 			(effects (font (size 1.27 1.27)) (hide yes))
 		)
-		(property "LCSC" "C7434207"
+		(property "LCSC" "C47773"
 			(at 435.6100 231.1400 0)
 			(effects (font (size 1.27 1.27)) (hide yes))
@@
 			(effects (font (size 1.27 1.27)))
 		)
-		(property "Value" "100nF"
+		(property "Value" "0.1uF"
 			(at 286.5120 275.5900 0)
 			(effects (font (size 1.27 1.27)))
@@
 			(effects (font (size 1.27 1.27)))
 		)
-		(property "Value" "0.1uF"
+		(property "Value" "10pF"
 			(at 535.4320 189.2300 0)
 			(effects (font (size 1.27 1.27)))
@@
 			(effects (font (size 1.27 1.27)) (hide yes))
 		)
-		(property "LCSC" "C1525"
+		(property "LCSC" "C32949"
 			(at 508.0000 231.1400 0)
 			(effects (font (size 1.27 1.27)) (hide yes))
@@
 			(effects (font (size 1.27 1.27)) (hide yes))
 		)
-		(property "LCSC" "C2013978"
+		(property "LCSC" "C424662"
 			(at 209.5500 306.0700 0)
 			(effects (font (size 1.27 1.27)) (hide yes))
